File: VXO7803-500-M.sch (KiCad schematic (older format))
At the start: 3 parts

Commit message: combined libraries
Parts:
- PS1: symbol VXO7803-500-M:VXO7803-500-M -> SIB_Footprint:VXO7803-500-M
Changed lines of the file:
@@
 $EndDescr
 $Comp
-L VXO7803-500-M:VXO7803-500-M PS1
+L SIB_Footprint:VXO7803-500-M PS1
 U 1 1 5ED341D9
 P 5500 3350

Commit message: changed cap footprint
Parts:
- C36: value 22uf 50V -> 22uf 10V; footprint Capacitor_SMD:C_0603_1608Metric -> Capacitor_SMD:C_1206_3216Metric
Changed lines of the file:
@@
 EESchema Schematic File Version 4
+LIBS:aducm_board-cache
 EELAYER 26 0
 EELAYER END
@@
 P 6700 3400
 F 0 "C36" H 6878 3446 50  0000 L CNN
-F 1 "22uf 50V" H 6878 3355 50  0000 L CNN
-F 2 "Capacitor_SMD:C_0603_1608Metric" H 6700 3400 50  0001 C CNN
+F 1 "22uf 10V" H 6878 3355 50  0000 L CNN
+F 2 "Capacitor_SMD:C_1206_3216Metric" H 6700 3400 50  0001 C CNN
 F 3 "~" H 6700 3400 50  0001 C CNN
 	1    6700 3400

Commit message: added footprint pa4318
Parts:
- added C37: 22uf 10V, Capacitor_SMD:C_1206_3216Metric, symbol pspice:CAP
- added L1: 10-47uF .5A, SIB_Generic:PA4318, symbol Device:L
Connections:
- wire segments 10 -> 14
Changed lines of the file:
@@
 Text HLabel 3800 3150 0    50   Input ~ 0
 +VIN
-Text HLabel 6950 3150 2    50   Output ~ 0
+Text HLabel 8800 3150 2    50   Output ~ 0
 +VOUT
 Text HLabel 4800 3350 0    50   Input ~ 0
@@
 	3800 3150 4050 3150
 Connection ~ 4050 3150
-Wire Wire Line
-	6700 3150 6950 3150
-Connection ~ 6700 3150
 Wire Wire Line
 	4050 3650 4050 3800
@@
 	4050 3800 3800 3800
 Connection ~ 4050 3800
+$Comp
+L Device:L L1
+U 1 1 5ED5FAEA
+P 7400 3150
+F 0 "L1" V 7222 3150 50  0000 C CNN
+F 1 "10-47uF .5A" V 7313 3150 50  0000 C CNN
+F 2 "SIB_Generic:PA4318" H 7400 3150 50  0001 C CNN
+F 3 "~" H 7400 3150 50  0001 C CNN
+	1    7400 3150
+	0    1    1    0
+$EndComp
+$Comp
+L pspice:CAP C37
+U 1 1 5ED5FB6C
+P 8000 3400
+F 0 "C37" H 8178 3446 50  0000 L CNN
+F 1 "22uf 10V" H 8178 3355 50  0000 L CNN
+F 2 "Capacitor_SMD:C_1206_3216Metric" H 8000 3400 50  0001 C CNN
+F 3 "~" H 8000 3400 50  0001 C CNN
+	1    8000 3400
+	1    0    0    -1
+$EndComp
+Wire Wire Line
+	6700 3150 7250 3150
+Connection ~ 6700 3150
+Wire Wire Line
+	7550 3150 8000 3150
+Wire Wire Line
+	8000 3150 8800 3150
+Connection ~ 8000 3150
+Wire Wire Line
+	8000 3650 8000 3800
+Wire Wire Line
+	8000 3800 6700 3800
+Connection ~ 6700 3800
 $EndSCHEMATC

Commit message: beginning layout
Parts:
- L1: value 10-47uF .5A -> 10-47uH .5A
- PS1: footprint SIB_Generic:CONV_VXO7803-500-M -> CONV_VXO7803-500-M
Changed lines of the file:
@@
 EESchema Schematic File Version 4
+LIBS:aducm_board-cache
 EELAYER 30 0
 EELAYER END
@@
 F 0 "PS1" H 5500 3817 50  0000 C CNN
 F 1 "VXO7803-500-M" H 5500 3726 50  0000 C CNN
-F 2 "SIB_Generic:CONV_VXO7803-500-M" H 5500 3350 50  0001 L BNN
+F 2 "CONV_VXO7803-500-M" H 5500 3350 50  0001 L BNN
 F 3 "3.5 mm" H 5500 3350 50  0001 L BNN
 F 4 "Manufacturer Recommendations" H 5500 3350 50  0001 L BNN "Field4"
@@
 U 1 1 5ED5FAEA
 P 7400 3150
+AR Path="/5ED209B3/5ED5FAEA" Ref="L1"  Part="1"
+AR Path="/5ED5FAEA" Ref="L1"  Part="1"
 F 0 "L1" V 7222 3150 50  0000 C CNN
-F 1 "10-47uF .5A" V 7313 3150 50  0000 C CNN
+F 1 "10-47uH .5A" V 7313 3150 50  0000 C CNN
 F 2 "SIB_Generic:PA4318" H 7400 3150 50  0001 C CNN
 F 3 "~" H 7400 3150 50  0001 C CNN

Commit message: added 3d model to molex connector. moved castle placement
Parts:
- PS1: footprint CONV_VXO7803-500-M -> SIB_Generic:CONV_VXO7803-500-M
Changed lines of the file:
@@
 F 0 "PS1" H 5500 3817 50  0000 C CNN
 F 1 "VXO7803-500-M" H 5500 3726 50  0000 C CNN
-F 2 "CONV_VXO7803-500-M" H 5500 3350 50  0001 L BNN
+F 2 "SIB_Generic:CONV_VXO7803-500-M" H 5500 3350 50  0001 L BNN
 F 3 "3.5 mm" H 5500 3350 50  0001 L BNN
 F 4 "Manufacturer Recommendations" H 5500 3350 50  0001 L BNN "Field4"
